File: PCB/hackpad.kicad_sch (KiCad schematic)
At the start: 34 parts, among them J1 OLED_128x64, K1 SW_Push, K2 SW_Push, K3 SW_Push, K4 SW_Push, Q1 SW_Push, T1 SW_Push, U1 XIAO-RP2040-DIP

Commit message: asd
Connections:
- net Column 1: now also U1.1 (GPIO26/ADC0/A0); no longer U1.5 (GPIO6/SDA)
- net Column 2: now also U1.2 (GPIO27/ADC1/A1); no longer U1.6 (GPIO7/SCL)
- net at J1.4 (SDA): now also U1.5 (GPIO6/SDA); no longer U1.1 (GPIO26/ADC0/A0)
- net at J1.3 (SCL): now also U1.6 (GPIO7/SCL); no longer U1.2 (GPIO27/ADC1/A1)
Changed lines of the file:
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@@
-	(wire
-		(pts
-			(xy 134.62 123.19) (xy 138.43 127)
-		)
-		(stroke
-			(width 0)
-			(type default)
-		)
-	)
 	(wire
 		(pts
@@
 	(wire
 		(pts
+			(xy 187.96 114.3) (xy 125.73 114.3)
+		)
+		(stroke
+			(width 0)
+			(type default)
+		)
+	)
+	(wire
+		(pts
 			(xy 90.17 148.59) (xy 105.41 148.59)
 		)
@@
 	(wire
 		(pts
-			(xy 191.77 111.76) (xy 142.24 111.76)
-		)
-		(stroke
-			(width 0)
-			(type default)
-		)
-	)
-	(wire
-		(pts
 			(xy 85.09 130.81) (xy 85.09 152.4)
 		)
@@
 	(wire
 		(pts
-			(xy 139.7 116.84) (xy 144.78 121.92)
+			(xy 191.77 111.76) (xy 129.54 111.76)
 		)
 		(stroke
@@
 	(wire
 		(pts
-			(xy 139.7 114.3) (xy 139.7 116.84)
-		)
-		(stroke
-			(width 0)
-			(type default)
-		)
-	)
-	(wire
-		(pts
 			(xy 69.85 87.63) (xy 69.85 109.22)
 		)
@@
 	(wire
 		(pts
-			(xy 187.96 114.3) (xy 143.51 114.3)
-		)
-		(stroke
-			(width 0)
-			(type default)
-		)
-	)
-	(wire
-		(pts
 			(xy 69.85 87.63) (xy 74.93 87.63)
 		)
@@
 	(wire
 		(pts
-			(xy 134.62 123.19) (xy 143.51 114.3)
-		)
-		(stroke
-			(width 0)
-			(type default)
-		)
-	)
-	(wire
-		(pts
-			(xy 138.43 127) (xy 143.51 127)
-		)
-		(stroke
-			(width 0)
-			(type default)
-		)
-	)
-	(wire
-		(pts
 			(xy 100.33 87.63) (xy 105.41 87.63)
 		)
@@
 	(wire
 		(pts
-			(xy 142.24 111.76) (xy 139.7 114.3)
-		)
-		(stroke
-			(width 0)
-			(type default)
-		)
-	)
-	(wire
-		(pts
 			(xy 100.33 130.81) (xy 100.33 152.4)
 		)
@@
 	(wire
 		(pts
+			(xy 125.73 114.3) (xy 125.73 140.97)
+		)
+		(stroke
+			(width 0)
+			(type default)
+		)
+	)
+	(wire
+		(pts
 			(xy 59.69 170.18) (xy 74.93 170.18)
 		)
@@
 	(wire
 		(pts
+			(xy 129.54 137.16) (xy 144.78 137.16)
+		)
+		(stroke
+			(width 0)
+			(type default)
+		)
+	)
+	(wire
+		(pts
 			(xy 74.93 105.41) (xy 90.17 105.41)
 		)
@@
 	(wire
 		(pts
+			(xy 129.54 111.76) (xy 129.54 137.16)
+		)
+		(stroke
+			(width 0)
+			(type default)
+		)
+	)
+	(wire
+		(pts
 			(xy 85.09 87.63) (xy 90.17 87.63)
 		)
@@
 	(wire
 		(pts
-			(xy 143.51 127) (xy 144.78 125.73)
+			(xy 125.73 140.97) (xy 144.78 140.97)
 		)
 		(stroke
@@
 	(global_label "Column 1"
 		(shape input)
-		(at 144.78 137.16 180)
+		(at 144.78 121.92 180)
 		(fields_autoplaced yes)
 		(effects
@@
 		)
 		(property "Intersheetrefs" "${INTERSHEET_REFS}"
-			(at 132.5422 137.16 0)
+			(at 132.5422 121.92 0)
 			(effects
 				(font
@@
 	(global_label "Column 2"
 		(shape input)
-		(at 144.78 140.97 180)
+		(at 144.78 125.73 180)
 		(fields_autoplaced yes)
 		(effects
@@
 		)
 		(property "Intersheetrefs" "${INTERSHEET_REFS}"
-			(at 132.5422 140.97 0)
-			(effects
-				(font
+			(at 132.5422 125.73 0)
+			(effects
+				(font
